File: Kicad/Samlet Racerbil/Samlet Racerbil.kicad_sch (KiCad schematic)
At the start: 8 parts

Commit message: Fix
Parts:
- Q?: value TIP120 -> (none)
Changed lines of the file:
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@@
       (effects (font (size 1.27 1.27)) (justify left))
     )
-    (property "Value" "TIP120" (id 1) (at 133.35 49.5299 0)
+    (property "Value" "" (id 1) (at 133.35 49.5299 0)
       (effects (font (size 1.27 1.27)) (justify left))
     )
@@
     )
     (path "/8fbfd03f-7055-40be-9db8-bb014db089a4"
-      (reference "Q?") (unit 1) (value "TIP120") (footprint "Package_TO_SOT_THT:TO-220-3_Vertical")
+      (reference "Q?") (unit 1) (value "IRL1404") (footprint "Package_TO_SOT_THT:TO-220-3_Vertical")
     )
     (path "/41d8c1d5-4b35-4e3a-ba04-bac7e10b12eb"
