File: Kicad/Controller/Controller.kicad_pcb (KiCad board)
At the start: 2 copper layers, 7 parts

Commit message: Update
Parts:
- removed 5V1: Connector, Connector_PinHeader_1.00mm:PinHeader_1x01_P1.00mm_Vertical
- removed ACC1, LDR1, PWM1: Conn_01x01_Female, Connector_PinHeader_1.00mm:PinHeader_1x01_P1.00mm_Vertical
- removed Ground1: Ground forbindelse, Connector_PinHeader_1.00mm:PinHeader_1x01_P1.00mm_Vertical
- added J1: Conn_01x06_Female, Connector_PinHeader_1.00mm:PinHeader_1x06_P1.00mm_Vertical, F.Cu at (115.3, 102.9)
- moved Pickit-forbindelse1 16.6 mm to (120.7, 113.0)
- moved PIC16f684 16.1 mm to (108.5, 106.0)
Connections:
- PIC16f684 pad 14: Net-(PIC16f684-Pad14) -> Net-(Pickit-forbindelse1-Pad4)
- Pickit-forbindelse1 pad 4: unconnected-(Pickit-forbindelse1-Pad4) -> Net-(Pickit-forbindelse1-Pad4)
- Pickit-forbindelse1 pad 5: unconnected-(Pickit-forbindelse1-Pad5) -> Net-(PIC16f684-Pad1)
Routing:
- net Net-(PIC16f684-Pad4): track 0.00 -> 38.7 mm
- net Net-(PIC16f684-Pad1): track 0.00 -> 21.6 mm
- net Net-(PIC16f684-Pad8): track 0.00 -> 20.0 mm
- net Net-(PIC16f684-Pad9): track 0.00 -> 17.0 mm
- net Net-(PIC16f684-Pad5): track 0.00 -> 14.5 mm
- net Net-(Pickit-forbindelse1-Pad4): track 0.00 -> 10.9 mm
- net Net-(PIC16f684-Pad11): track 0.00 -> 5.20 mm
- net Net-(PIC16f684-Pad12): track 0.00 -> 4.56 mm

Commit message: Update Controller.kicad_pcb
Other:
- board text added: "Mongo Racing"
Changed lines of the file:
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@@
     )
+  )
+  (gr_text "Mongo Racing\n" (at 104.14 111.76 270) (layer "B.Cu")
+    (effects (font (size 1.5 1.5) (thickness 0.3)) (justify mirror))
   )
   (segment (start 114.266746 101.6) (end 115.3 102.633254) (width 0.5) (layer "B.Cu") (net 1))

Commit message: Update
Parts:
- removed PIC16f684: PIC16F684-IP, Package_DIP:DIP-14_W7.62mm_Socket
- removed Pickit-forbindelse1: Pickit forbindelse, Connector_PinHeader_1.00mm:PinHeader_1x06_P1.00mm_Vertical
- added J2: Conn_01x07_Female, Connector_PinHeader_1.00mm:PinHeader_1x07_P1.00mm_Vertical, F.Cu at (114.3, 107.7)
- added PIC16f1: PIC16F684-IP, Package_DIP:DIP-14_W7.62mm_Socket, F.Cu at (119.5, 97.1)
- added Pickit1: Conn_01x05_Female, Connector_PinHeader_1.00mm:PinHeader_1x05_P1.00mm_Vertical, F.Cu at (137.2, 102.3)
- J1: value Conn_01x06_Female -> Conn_01x07_Female; footprint Connector_PinHeader_1.00mm:PinHeader_1x06_P1.00mm_Vertical -> Connector_PinHeader_1.00mm:PinHeader_1x07_P1.00mm_Vertical
- moved J1 17.0 mm to (132.1, 99.9), turned to 0 degrees
Connections:
- J1 pad 6: unconnected-(J1-Pad6) -> Net-(J1-Pad6)
Routing:
- net Net-(J2-Pad1): track 0.00 -> 44.1 mm
- net Net-(PIC16f684-Pad4): track 38.7 -> 0.00 mm
- net Net-(J2-Pad5): track 0.00 -> 31.5 mm
- net Net-(J1-Pad4): track 20.0 -> 5.77 mm
- net Net-(J1-Pad1): track 21.6 -> 11.4 mm
- net Net-(J1-Pad7): track 0.00 -> 8.56 mm
- net Net-(J2-Pad2): track 0.00 -> 8.37 mm
- net Net-(J1-Pad5): track 14.5 -> 6.41 mm
- net Net-(J2-Pad3): track 0.00 -> 7.62 mm
- net Net-(J1-Pad6): track 0.00 -> 7.37 mm
- net Net-(J1-Pad3): track 17.0 -> 10.4 mm
- net Net-(J2-Pad4): track 0.00 -> 6.24 mm
- net Net-(J2-Pad7): track 0.00 -> 6.00 mm
- net Net-(J2-Pad6): track 0.00 -> 5.36 mm
- net Net-(PIC16f684-Pad11): track 5.20 -> 0.00 mm
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Other:
- board text removed: "Mongo Racing"

Commit message: Fix
Other:
- board text added: "MongoRacing"
Changed lines of the file:
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@@
     )
+  )
+  (gr_text "MongoRacing" (at 123.19 115.57 180) (layer "B.Cu")
+    (effects (font (size 1.5 1.5) (thickness 0.3)) (justify mirror))
   )
   (segment (start 129.33 97.12) (end 132.08 99.87) (width 0.7) (layer "B.Cu") (net 1))

Commit message: h
Parts:
- J1, J2: footprint Connector_PinHeader_1.00mm:PinHeader_1x07_P1.00mm_Vertical -> Connector_PinHeader_2.54mm:PinHeader_1x07_P2.54mm_Vertical
- Pickit1: footprint Connector_PinHeader_1.00mm:PinHeader_1x05_P1.00mm_Vertical -> Connector_PinHeader_2.54mm:PinHeader_1x05_P2.54mm_Vertical
- moved J1 8.11 mm to (135.9, 92.7)
- moved Pickit1 6.82 mm to (142.2, 97.8)
- moved PIC16f1 5.79 mm to (123.2, 92.7)
- moved J2 4.73 mm to (118.1, 110.5)
Connections:
- net Net-(J1-Pad1) renamed Earth
Routing:
- net Net-(J2-Pad1): track 44.1 -> 55.8 mm
- net Net-(J1-Pad7): track 8.56 -> 5.07 mm
- net Net-(J2-Pad2): track 8.37 -> 5.09 mm
- net Net-(J2-Pad3): track 7.62 -> 5.09 mm
- net Net-(J1-Pad6): track 7.37 -> 5.07 mm
- net Net-(J1-Pad5): track 6.41 -> 5.07 mm
- net Net-(J2-Pad4): track 6.24 -> 5.09 mm
- net Net-(J1-Pad3): track 10.4 -> 11.4 mm
- net Net-(J2-Pad7): track 6.00 -> 5.09 mm
- net Net-(J1-Pad4): track 5.77 -> 5.07 mm
- net Net-(J1-Pad2): track 10.8 -> 11.4 mm
- added copper zone on B.Cu, net Earth
