File: Kicad/Controller/Controller.kicad_sch (KiCad schematic)
At the start: 7 parts

Commit message: Update
Parts:
- removed 5V1: Connector, Connector_PinHeader_1.00mm:PinHeader_1x01_P1.00mm_Vertical, symbol Connector:Conn_01x01_Female
- removed ACC1, LDR1, PWM1: Conn_01x01_Female, Connector_PinHeader_1.00mm:PinHeader_1x01_P1.00mm_Vertical, symbol Connector:Conn_01x01_Female
- removed Ground1: Ground forbindelse, Connector_PinHeader_1.00mm:PinHeader_1x01_P1.00mm_Vertical, symbol Connector:Conn_01x01_Female
- added J1: (no value), symbol Connector:Conn_01x06_Female
- PIC16f684: footprint (none) -> Package_DIP:DIP-14_W7.62mm_Socket
Connections:
- net at Pickit-forbindelse1.4 (Pin_4): now also PIC16f684.14 (VSS), J1.2 (Pin_2)
- net at Pickit-forbindelse1.5 (Pin_5): now also PIC16f684.1 (VDD), J1.1 (Pin_1)
- net at PIC16f684.5 (P1A/CCP1/RC5): now also J1.5 (Pin_5)
- net at PIC16f684.9 (C2IN-/AN5/RC1): now also J1.3 (Pin_3)
- net at PIC16f684.8 (P1D/AN6/RC2): now also J1.4 (Pin_4)
Other:
- note added: "ACC"
- note added: "LDR"
- note added: "PWM"
Changed lines of the file:
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@@
 (kicad_sch (version 20211123) (generator eeschema)
   (paper "A4")
+  (junction (at 139.7 111.76) (diameter 0) (color 0 0 0 0)
+  )
+  (junction (at 139.7 74.93) (diameter 0) (color 0 0 0 0)
+  )
+  (wire (pts (xy 68.58 88.9) (xy 76.2 88.9))
+    (stroke (width 0) (type default) (color 0 0 0 0))
+  )
   (wire (pts (xy 68.58 86.36) (xy 82.55 86.36))
     (stroke (width 0) (type default) (color 0 0 0 0))
@@
     (stroke (width 0) (type default) (color 0 0 0 0))
   )
+  (wire (pts (xy 196.85 88.9) (xy 201.93 88.9))
+    (stroke (width 0) (type default) (color 0 0 0 0))
+  )
+  (wire (pts (xy 195.58 88.9) (xy 195.58 91.44))
+    (stroke (width 0) (type default) (color 0 0 0 0))
+  )
   (wire (pts (xy 82.55 86.36) (xy 82.55 93.98))
+    (stroke (width 0) (type default) (color 0 0 0 0))
+  )
+  (wire (pts (xy 198.12 96.52) (xy 201.93 96.52))
     (stroke (width 0) (type default) (color 0 0 0 0))
   )
@@
     (stroke (width 0) (type default) (color 0 0 0 0))
   )
-  (wire (pts (xy 180.34 88.9) (xy 189.23 88.9))
+  (wire (pts (xy 180.34 88.9) (xy 195.58 88.9))
     (stroke (width 0) (type default) (color 0 0 0 0))
   )
-  (wire (pts (xy 180.34 91.44) (xy 189.23 91.44))
+  (wire (pts (xy 193.04 93.98) (xy 201.93 93.98))
+    (stroke (width 0) (type default) (color 0 0 0 0))
+  )
+  (wire (pts (xy 139.7 111.76) (xy 196.85 111.76))
     (stroke (width 0) (type default) (color 0 0 0 0))
   )
   (wire (pts (xy 139.7 74.93) (xy 139.7 78.74))
+    (stroke (width 0) (type default) (color 0 0 0 0))
+  )
+  (wire (pts (xy 180.34 91.44) (xy 193.04 91.44))
+    (stroke (width 0) (type default) (color 0 0 0 0))
+  )
+  (wire (pts (xy 195.58 91.44) (xy 201.93 91.44))
+    (stroke (width 0) (type default) (color 0 0 0 0))
+  )
+  (wire (pts (xy 139.7 74.93) (xy 201.93 74.93))
     (stroke (width 0) (type default) (color 0 0 0 0))
   )
@@
     (stroke (width 0) (type default) (color 0 0 0 0))
   )
+  (wire (pts (xy 76.2 74.93) (xy 139.7 74.93))
+    (stroke (width 0) (type default) (color 0 0 0 0))
+  )
   (wire (pts (xy 68.58 93.98) (xy 78.74 93.98))
     (stroke (width 0) (type default) (color 0 0 0 0))
@@
     (stroke (width 0) (type default) (color 0 0 0 0))
   )
+  (wire (pts (xy 193.04 91.44) (xy 193.04 93.98))
+    (stroke (width 0) (type default) (color 0 0 0 0))
+  )
+  (wire (pts (xy 201.93 74.93) (xy 201.93 86.36))
+    (stroke (width 0) (type default) (color 0 0 0 0))
+  )
+  (wire (pts (xy 74.93 91.44) (xy 74.93 111.76))
+    (stroke (width 0) (type default) (color 0 0 0 0))
+  )
   (wire (pts (xy 68.58 96.52) (xy 83.82 96.52))
     (stroke (width 0) (type default) (color 0 0 0 0))
   )
-  (wire (pts (xy 180.34 99.06) (xy 186.69 99.06))
+  (wire (pts (xy 198.12 99.06) (xy 198.12 96.52))
     (stroke (width 0) (type default) (color 0 0 0 0))
+  )
+  (wire (pts (xy 68.58 91.44) (xy 74.93 91.44))
+    (stroke (width 0) (type default) (color 0 0 0 0))
+  )
+  (wire (pts (xy 74.93 111.76) (xy 139.7 111.76))
+    (stroke (width 0) (type default) (color 0 0 0 0))
+  )
+  (wire (pts (xy 180.34 99.06) (xy 198.12 99.06))
+    (stroke (width 0) (type default) (color 0 0 0 0))
+  )
+  (wire (pts (xy 196.85 111.76) (xy 196.85 88.9))
+    (stroke (width 0) (type default) (color 0 0 0 0))
+  )
+  (wire (pts (xy 76.2 88.9) (xy 76.2 74.93))
+    (stroke (width 0) (type default) (color 0 0 0 0))
+  )
+  (text "ACC\n" (at 207.01 92.71 0)
+    (effects (font (size 1.27 1.27)) (justify left bottom))
+  )
+  (text "LDR\n" (at 207.01 95.25 0)
+    (effects (font (size 1.27 1.27)) (justify left bottom))
+  )
+  (text "PWM\n" (at 207.01 97.79 0)
+    (effects (font (size 1.27 1.27)) (justify left bottom))
   )
   (text "TJek om de er korrekt forbundet" (at 63.5 80.01 0)
@@
     (pin "6")
   )
-  (symbol (lib_id "Connector:Conn_01x01_Female") (at 139.7 116.84 270) (unit 1)
+  (symbol (lib_id "Connector:Conn_01x06_Female") (at 207.01 91.44 0) (unit 1)
     (in_bom yes) (on_board yes) (fields_autoplaced)
-    (property "Reference" "Ground1" (id 0) (at 140.97 116.2049 90)
+    (property "Reference" "J1" (id 0) (at 208.28 92.7099 0)
       (effects (font (size 1.27 1.27)) (justify left))
     )
-    (property "Value" "Ground forbindelse" (id 1) (at 140.97 117.4749 90)
+    (property "Value" "" (id 1) (at 208.28 93.9799 0)
       (effects (font (size 1.27 1.27)) (justify left) hide)
     )
-    (property "Footprint" "Connector_PinHeader_1.00mm:PinHeader_1x01_P1.00mm_Vertical" (id 2) (at 139.7 116.84 0)
+    (property "Footprint" "" (id 2) (at 207.01 91.44 0)
       (effects (font (size 1.27 1.27)) hide)
     )
-    (property "Datasheet" "~" (id 3) (at 139.7 116.84 0)
+    (property "Datasheet" "~" (id 3) (at 207.01 91.44 0)
       (effects (font (size 1.27 1.27)) hide)
     )
     (pin "1")
-  )
-  (symbol (lib_id "Connector:Conn_01x01_Female") (at 191.77 99.06 0) (unit 1)
-    (in_bom yes) (on_board yes) (fields_autoplaced)
-    (property "Reference" "PWM1" (id 0) (at 193.04 99.0599 0)
-      (effects (font (size 1.27 1.27)) (justify left))
-    )
-    (property "Value" "Conn_01x01_Female" (id 1) (at 193.04 100.3299 0)
-      (effects (font (size 1.27 1.27)) (justify left) hide)
-    )
-    (property "Footprint" "Connector_PinHeader_1.00mm:PinHeader_1x01_P1.00mm_Vertical" (id 2) (at 191.77 99.06 0)
-      (effects (font (size 1.27 1.27)) hide)
-    )
-    (property "Datasheet" "~" (id 3) (at 191.77 99.06 0)
-      (effects (font (size 1.27 1.27)) hide)
-    )
-    (pin "1")
-  )
-  (symbol (lib_id "Connector:Conn_01x01_Female") (at 194.31 88.9 0) (unit 1)
-    (in_bom yes) (on_board yes) (fields_autoplaced)
-    (property "Reference" "ACC1" (id 0) (at 195.58 88.8999 0)
-      (effects (font (size 1.27 1.27)) (justify left))
-    )
-    (property "Value" "Conn_01x01_Female" (id 1) (at 195.58 90.1699 0)
-      (effects (font (size 1.27 1.27)) (justify left) hide)
-    )
-    (property "Footprint" "Connector_PinHeader_1.00mm:PinHeader_1x01_P1.00mm_Vertical" (id 2) (at 194.31 88.9 0)
-      (effects (font (size 1.27 1.27)) hide)
-    )
-    (property "Datasheet" "~" (id 3) (at 194.31 88.9 0)
-      (effects (font (size 1.27 1.27)) hide)
-    )
-    (pin "1")
-  )
-  (symbol (lib_id "Connector:Conn_01x01_Female") (at 139.7 69.85 90) (unit 1)
-    (in_bom yes) (on_board yes) (fields_autoplaced)
-    (property "Reference" "5V1" (id 0) (at 140.97 70.4849 90)
-      (effects (font (size 1.27 1.27)) (justify right))
-    )
-    (property "Value" "Connector" (id 1) (at 140.97 71.7549 90)
-      (effects (font (size 1.27 1.27)) (justify right) hide)
-    )
-    (property "Footprint" "Connector_PinHeader_1.00mm:PinHeader_1x01_P1.00mm_Vertical" (id 2) (at 139.7 69.85 0)
-      (effects (font (size 1.27 1.27)) hide)
-    )
-    (property "Datasheet" "~" (id 3) (at 139.7 69.85 0)
-      (effects (font (size 1.27 1.27)) hide)
-    )
-    (pin "1")
+    (pin "2")
+    (pin "3")
+    (pin "4")
+    (pin "5")
+    (pin "6")
   )
   (symbol (lib_id "MCU_Microchip_PIC16:PIC16F684-IP") (at 139.7 93.98 0) (unit 1)
@@
       (effects (font (size 1.27 1.27)) (justify left) hide)
     )
-    (property "Footprint" "" (id 2) (at 139.7 93.98 0)
+    (property "Footprint" "Package_DIP:DIP-14_W7.62mm_Socket" (id 2) (at 139.7 93.98 0)
       (effects (font (size 1.27 1.27)) hide)
     )
@@
     (pin "9")
   )
-  (symbol (lib_id "Connector:Conn_01x01_Female") (at 194.31 91.44 0) (unit 1)
-    (in_bom yes) (on_board yes) (fields_autoplaced)
-    (property "Reference" "LDR1" (id 0) (at 195.58 91.4399 0)
-      (effects (font (size 1.27 1.27)) (justify left))
-    )
-    (property "Value" "Conn_01x01_Female" (id 1) (at 195.58 92.7099 0)
-      (effects (font (size 1.27 1.27)) (justify left) hide)
-    )
-    (property "Footprint" "Connector_PinHeader_1.00mm:PinHeader_1x01_P1.00mm_Vertical" (id 2) (at 194.31 91.44 0)
-      (effects (font (size 1.27 1.27)) hide)
-    )
-    (property "Datasheet" "~" (id 3) (at 194.31 91.44 0)
-      (effects (font (size 1.27 1.27)) hide)
-    )
-    (pin "1")
-  )
   (sheet_instances
     (path "/" (page "1"))
   )
   (symbol_instances
-    (path "/be8050df-c3dd-4998-9fc4-ed0ab9ca33c2"
-      (reference "5V1") (unit 1) (value "Connector") (footprint "Connector_PinHeader_1.00mm:PinHeader_1x01_P1.00mm_Vertical")
-    )
-    (path "/92e22236-bf4b-4a77-8ff3-2e3a4fd5f7ad"
-      (reference "ACC1") (unit 1) (value "Conn_01x01_Female") (footprint "Connector_PinHeader_1.00mm:PinHeader_1x01_P1.00mm_Vertical")
-    )
-    (path "/662b796f-b530-402b-9af2-84a3224320fa"
-      (reference "Ground1") (unit 1) (value "Ground forbindelse") (footprint "Connector_PinHeader_1.00mm:PinHeader_1x01_P1.00mm_Vertical")
-    )
-    (path "/f8cee974-2385-448d-a979-24059f2eccf1"
-      (reference "LDR1") (unit 1) (value "Conn_01x01_Female") (footprint "Connector_PinHeader_1.00mm:PinHeader_1x01_P1.00mm_Vertical")
+    (path "/754700b8-82bc-4d0e-926c-196988658878"
+      (reference "J1") (unit 1) (value "Conn_01x06_Female") (footprint "Connector_PinHeader_1.00mm:PinHeader_1x06_P1.00mm_Vertical")
     )
     (path "/e6156301-a13c-4626-8405-1e6dde4c94e4"
       (reference "PIC16f684") (unit 1) (value "PIC16F684-IP") (footprint "Package_DIP:DIP-14_W7.62mm_Socket")
     )
-    (path "/8658435a-3281-44ea-988c-393a06d9e1ab"
-      (reference "PWM1") (unit 1) (value "Conn_01x01_Female") (footprint "Connector_PinHeader_1.00mm:PinHeader_1x01_P1.00mm_Vertical")
-    )
     (path "/1603a895-44dd-40ac-b205-4924d6c37b4b"

Commit message: Update
Parts:
- removed J1: (no value), symbol Connector:Conn_01x06_Female
- removed PIC16f684: PIC16F684-IP, Package_DIP:DIP-14_W7.62mm_Socket, symbol MCU_Microchip_PIC16:PIC16F684-IP
- removed Pickit-forbindelse1: Pickit forbindelse, Connector_PinHeader_1.00mm:PinHeader_1x06_P1.00mm_Vertical, symbol Connector:Conn_01x06_Female
- added J1, J2: Conn_01x07_Female, Connector_PinHeader_1.00mm:PinHeader_1x07_P1.00mm_Vertical, symbol Connector:Conn_01x07_Female
- added PIC16f1: PIC16F684-IP, Package_DIP:DIP-14_W7.62mm_Socket, symbol MCU_Microchip_PIC16:PIC16F684-IP
- added Pickit1: Conn_01x05_Female, Connector_PinHeader_1.00mm:PinHeader_1x05_P1.00mm_Vertical, symbol Connector:Conn_01x05_Female
Connections:
- new net: J1.1 (Pin_1), PIC16f1.14 (VSS), Pickit1.3 (Pin_3)
- new net: J1.2 (Pin_2), PIC16f1.13 (RA0/AN0/C1IN+/ICSPDAT/ULPWU), Pickit1.2 (Pin_2)
- new net: J1.3 (Pin_3), PIC16f1.12 (RA1/AN1/C1IN-/Vref/ICSPCLK), Pickit1.1 (Pin_1)
- new net: J1.4 (Pin_4), PIC16f1.11 (RA2/AN2/T0CKI/INT/C1OUT)
- new net: J1.5 (Pin_5), PIC16f1.10 (C2IN+/AN4/RC0)
- new net: J1.6 (Pin_6), PIC16f1.9 (C2IN-/AN5/RC1)
- new net: J1.7 (Pin_7), PIC16f1.8 (P1D/AN6/RC2)
- new net: J2.1 (Pin_1), PIC16f1.1 (VDD), Pickit1.4 (Pin_4)
- new net: J2.7 (Pin_7), PIC16f1.2 (RA5/T1CKI/OSC1/CLKIN)
- new net: J2.6 (Pin_6), PIC16f1.3 (RA4/AN3/~{T1G}/OSC2/CLKOUT)
- new net: J2.5 (Pin_5), PIC16f1.4 (RA3/~{MCLR}/Vpp), Pickit1.5 (Pin_5)
- new net: J2.4 (Pin_4), PIC16f1.5 (P1A/CCP1/RC5)
- new net: J2.3 (Pin_3), PIC16f1.6 (P1B/C2OUT/RC4)
- new net: J2.2 (Pin_2), PIC16f1.7 (P1C/AN7/RC3)
Other:
- note removed: "ACC"
- note removed: "LDR"
- note removed: "PWM"
- note removed: "TJek om de er korrekt forbundet"

Commit message: h
Parts:
- J1, J2: value Conn_01x07_Female -> (none); footprint Connector_PinHeader_1.00mm:PinHeader_1x07_P1.00mm_Vertical -> (none)
- Pickit1: value Conn_01x05_Female -> (none); footprint Connector_PinHeader_1.00mm:PinHeader_1x05_P1.00mm_Vertical -> (none)
Connections:
- net Earth: now reaches J1.1 (Pin_1), PIC16f1.14 (VSS), Pickit1.3 (Pin_3)
Changed lines of the file:
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@@
   (junction (at 148.59 82.55) (diameter 0) (color 0 0 0 0)
   )
+  (junction (at 151.13 120.65) (diameter 0) (color 0 0 0 0)
+  )
   (junction (at 148.59 132.08) (diameter 0) (color 0 0 0 0)
   )
@@
   )
   (wire (pts (xy 148.59 143.51) (xy 96.52 143.51))
+    (stroke (width 0) (type default) (color 0 0 0 0))
+  )
+  (wire (pts (xy 151.13 120.65) (xy 151.13 121.92))
     (stroke (width 0) (type default) (color 0 0 0 0))
   )
@@
     (in_bom yes) (on_board yes) (fields_autoplaced)
     (property "Reference" "J1" (id 0) (at 151.13 74.93 90))
-    (property "Value" "Conn_01x07_Female" (id 1) (at 161.29 78.105 0)
-      (effects (font (size 1.27 1.27)) hide)
-    )
-    (property "Footprint" "Connector_PinHeader_1.00mm:PinHeader_1x07_P1.00mm_Vertical" (id 2) (at 151.13 77.47 0)
+    (property "Value" "" (id 1) (at 161.29 78.105 0)
+      (effects (font (size 1.27 1.27)) hide)
+    )
+    (property "Footprint" "" (id 2) (at 151.13 77.47 0)
       (effects (font (size 1.27 1.27)) hide)
     )
@@
     (pin "9")
   )
+  (symbol (lib_id "power:Earth") (at 151.13 121.92 0) (unit 1)
+    (in_bom yes) (on_board yes) (fields_autoplaced)
+    (property "Reference" "#PWR?" (id 0) (at 151.13 128.27 0)
+      (effects (font (size 1.27 1.27)) hide)
+    )
+    (property "Value" "Earth" (id 1) (at 151.13 125.73 0)
+      (effects (font (size 1.27 1.27)) hide)
+    )
+    (property "Footprint" "" (id 2) (at 151.13 121.92 0)
+      (effects (font (size 1.27 1.27)) hide)
+    )
+    (property "Datasheet" "~" (id 3) (at 151.13 121.92 0)
+      (effects (font (size 1.27 1.27)) hide)
+    )
+    (pin "1")
+  )
   (symbol (lib_id "Connector:Conn_01x07_Female") (at 151.13 137.16 270) (unit 1)
     (in_bom yes) (on_board yes) (fields_autoplaced)
     (property "Reference" "J2" (id 0) (at 151.13 139.7 90))
-    (property "Value" "Conn_01x07_Female" (id 1) (at 140.97 136.525 0)
-      (effects (font (size 1.27 1.27)) hide)
-    )
-    (property "Footprint" "Connector_PinHeader_1.00mm:PinHeader_1x07_P1.00mm_Vertical" (id 2) (at 151.13 137.16 0)
+    (property "Value" "" (id 1) (at 140.97 136.525 0)
+      (effects (font (size 1.27 1.27)) hide)
+    )
+    (property "Footprint" "" (id 2) (at 151.13 137.16 0)
       (effects (font (size 1.27 1.27)) hide)
     )
@@
     (in_bom yes) (on_board yes) (fields_autoplaced)
     (property "Reference" "Pickit1" (id 0) (at 83.185 93.98 0))
-    (property "Value" "Conn_01x05_Female" (id 1) (at 83.185 93.98 0)
-      (effects (font (size 1.27 1.27)) hide)
-    )
-    (property "Footprint" "Connector_PinHeader_1.00mm:PinHeader_1x05_P1.00mm_Vertical" (id 2) (at 82.55 101.6 0)
+    (property "Value" "" (id 1) (at 83.185 93.98 0)
+      (effects (font (size 1.27 1.27)) hide)
+    )
+    (property "Footprint" "" (id 2) (at 82.55 101.6 0)
       (effects (font (size 1.27 1.27)) hide)
     )
@@
   )
   (symbol_instances
+    (path "/c38f28b6-5bd4-4cf9-b273-1e7b230f6b42"
+      (reference "#PWR?") (unit 1) (value "Earth") (footprint "")
+    )
     (path "/9a5b1e93-c412-45a8-9f57-8617c0a9ea62"
-      (reference "J1") (unit 1) (value "Conn_01x07_Female") (footprint "Connector_PinHeader_1.00mm:PinHeader_1x07_P1.00mm_Vertical")
+      (reference "J1") (unit 1) (value "Conn_01x07_Female") (footprint "Connector_PinHeader_2.54mm:PinHeader_1x07_P2.54mm_Vertical")
     )
     (path "/d1b39b6e-1a47-41b4-8b5e-1b1d883811c8"
-      (reference "J2") (unit 1) (value "Conn_01x07_Female") (footprint "Connector_PinHeader_1.00mm:PinHeader_1x07_P1.00mm_Vertical")
+      (reference "J2") (unit 1) (value "Conn_01x07_Female") (footprint "Connector_PinHeader_2.54mm:PinHeader_1x07_P2.54mm_Vertical")
     )
     (path "/b06d44d7-e749-4b3e-a5a2-2aba241e3fea"
@@
     )
     (path "/d6bfb401-cf49-4615-8935-d7ae23ccae89"
-      (reference "Pickit1") (unit 1) (value "Conn_01x05_Female") (footprint "Connector_PinHeader_1.00mm:PinHeader_1x05_P1.00mm_Vertical")
-    )
-  )
+      (reference "Pickit1") (unit 1) (value "Conn_01x05_Female") (footprint "Connector_PinHeader_2.54mm:PinHeader_1x05_P2.54mm_Vertical")
+    )
+  )
