File: Kicad/Inputs/Inputs.kicad_pcb (KiCad board)
At the start: 2 copper layers, 5 parts

Commit message: Update
Parts:
- removed 5V: 5V, Connector_PinHeader_1.00mm:PinHeader_1x01_P1.00mm_Vertical
- removed Ground: Ground, Connector_PinHeader_1.00mm:PinHeader_1x01_P1.00mm_Vertical
- removed OUT: OUT, Connector_PinHeader_1.00mm:PinHeader_1x01_P1.00mm_Vertical
- added J1: 5V, Connector_PinHeader_1.00mm:PinHeader_1x02_P1.00mm_Vertical, F.Cu at (134.6, 82.5)
- added J2: GROUND, Connector_PinHeader_1.00mm:PinHeader_1x02_P1.00mm_Vertical, F.Cu at (142.2, 80.0)
- added J3: Conn_01x05_Female, Connector_PinHeader_1.00mm:PinHeader_1x05_P1.00mm_Vertical, F.Cu at (140.4, 82.5)
- added LDR-OUT1: LDR-OUT, Connector_PinHeader_1.00mm:PinHeader_1x01_P1.00mm_Vertical, F.Cu at (142.2, 83.8)
- moved R1 7.73 mm to (134.6, 86.4)
- moved R2 6.35 mm to (146.1, 83.8), turned to 90 degrees
Routing:
- net Net-(LDR-OUT1-Pad1): track 0.00 -> 6.35 mm
- net Net-(R2-Pad2): track 0.00 -> 3.98 mm
- net Net-(J2-Pad2): track 0.00 -> 2.88 mm
- net Net-(R1-Pad1): track 0.00 -> 2.81 mm
- net Net-(J1-Pad1): track 0.00 -> 1.81 mm

Commit message: Update
Changed lines of the file:
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@@
     )
   )
-  (segment (start 142.24 86.36) (end 142.24 83.82) (width 0.25) (layer "B.Cu") (net 1))
-  (segment (start 142.24 83.82) (end 146.05 83.82) (width 0.25) (layer "B.Cu") (net 1))
-  (segment (start 134.62 86.36) (end 134.62 83.55) (width 0.25) (layer "B.Cu") (net 2))
-  (segment (start 146.05 80.42) (end 142.65 80.42) (width 0.25) (layer "B.Cu") (net 3))
-  (segment (start 142.65 80.42) (end 142.24 80.01) (width 0.25) (layer "B.Cu") (net 3))
-  (segment (start 134.62 82.55) (end 136.43 82.55) (width 0.25) (layer "B.Cu") (net 4))
-  (segment (start 141.24 80.01) (end 141.24 81.74) (width 0.25) (layer "B.Cu") (net 5))
-  (segment (start 141.24 81.74) (end 140.43 82.55) (width 0.25) (layer "B.Cu") (net 5))
+  (segment (start 142.24 83.82) (end 146.05 83.82) (width 0.7) (layer "B.Cu") (net 1))
+  (segment (start 142.24 86.36) (end 142.24 83.82) (width 0.7) (layer "B.Cu") (net 1))
+  (segment (start 134.62 86.36) (end 134.62 83.55) (width 0.7) (layer "B.Cu") (net 2))
+  (segment (start 142.65 80.42) (end 142.24 80.01) (width 0.7) (layer "B.Cu") (net 3))
+  (segment (start 146.05 80.42) (end 142.65 80.42) (width 0.7) (layer "B.Cu") (net 3))
+  (segment (start 134.62 82.55) (end 136.43 82.55) (width 0.7) (layer "B.Cu") (net 4))
+  (segment (start 140.43 80.82) (end 141.24 80.01) (width 0.7) (layer "B.Cu") (net 5))
+  (segment (start 140.43 82.55) (end 140.43 80.82) (width 0.7) (layer "B.Cu") (net 5))
 )

Commit message: Fix
Parts:
- added J4: ACC OUT, Connector_PinHeader_1.00mm:PinHeader_1x01_P1.00mm_Vertical, F.Cu at (138.4, 80.0)
Connections:
- J3 pad 3: unconnected-(J3-Pad3) -> Net-(J3-Pad3)
Routing:
- net Net-(J3-Pad3): track 0.00 -> 2.54 mm
Changed lines of the file:
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@@
   (net 0 "")
   (net 1 "Net-(LDR-OUT1-Pad1)")
-  (net 2 "Net-(R1-Pad1)")
-  (net 3 "Net-(R2-Pad2)")
+  (net 2 "Net-(J1-Pad2)")
+  (net 3 "Net-(J2-Pad1)")
   (net 4 "Net-(J1-Pad1)")
   (net 5 "Net-(J2-Pad2)")
   (net 6 "unconnected-(J3-Pad2)")
-  (net 7 "unconnected-(J3-Pad3)")
+  (net 7 "Net-(J3-Pad3)")
   (net 8 "unconnected-(J3-Pad4)")
   (footprint "Connector_PinHeader_1.00mm:PinHeader_1x02_P1.00mm_Vertical" (layer "F.Cu")
@@
     (fp_line (start -0.635 1.5) (end -0.635 -0.1825) (layer "F.Fab") (width 0.1))
     (pad "1" thru_hole rect (at 0 0 270) (size 0.85 0.85) (drill 0.5) (layers *.Cu *.Mask)
-      (net 3 "Net-(R2-Pad2)") (pinfunction "Pin_1") (pintype "passive"))
+      (net 3 "Net-(J2-Pad1)") (pinfunction "Pin_1") (pintype "passive"))
     (pad "2" thru_hole oval (at 0 1 270) (size 0.85 0.85) (drill 0.5) (layers *.Cu *.Mask)
       (net 5 "Net-(J2-Pad2)") (pinfunction "Pin_2") (pintype "passive"))
@@
     (fp_line (start 0 0) (end 2.01 0) (layer "F.Fab") (width 0.1))
     (pad "1" thru_hole circle (at 0 0) (size 1.4 1.4) (drill 0.7) (layers *.Cu *.Mask)
-      (net 2 "Net-(R1-Pad1)") (pintype "passive"))
+      (net 2 "Net-(J1-Pad2)") (pintype "passive"))
     (pad "2" thru_hole oval (at 7.62 0) (size 1.4 1.4) (drill 0.7) (layers *.Cu *.Mask)
       (net 1 "Net-(LDR-OUT1-Pad1)") (pintype "passive"))
@@
       (net 6 "unconnected-(J3-Pad2)") (pinfunction "Pin_2") (pintype "passive"))
     (pad "3" thru_hole oval (at 0 2 270) (size 0.85 0.85) (drill 0.5) (layers *.Cu *.Mask)
-      (net 7 "unconnected-(J3-Pad3)") (pinfunction "Pin_3") (pintype "passive"))
+      (net 7 "Net-(J3-Pad3)") (pinfunction "Pin_3") (pintype "passive"))
     (pad "4" thru_hole oval (at 0 3 270) (size 0.85 0.85) (drill 0.5) (layers *.Cu *.Mask)
       (net 8 "unconnected-(J3-Pad4)") (pinfunction "Pin_4") (pintype "passive"))
@@
       (net 1 "Net-(LDR-OUT1-Pad1)") (pintype "passive"))
     (pad "2" thru_hole circle (at 3.4 0 90) (size 1.5 1.5) (drill 0.8) (layers *.Cu *.Mask)
-      (net 3 "Net-(R2-Pad2)") (pintype "passive"))
+      (net 3 "Net-(J2-Pad1)") (pintype "passive"))
     (model "${KICAD6_3DMODEL_DIR}/OptoDevice.3dshapes/R_LDR_5.1x4.3mm_P3.4mm_Vertical.wrl"
       (offset (xyz 0 0 0))
@@
     (pad "1" thru_hole rect (at 0 0) (size 0.85 0.85) (drill 0.5) (layers *.Cu *.Mask)
       (net 1 "Net-(LDR-OUT1-Pad1)") (pinfunction "Pin_1") (pintype "passive"))
+    (model "${KICAD6_3DMODEL_DIR}/Connector_PinHeader_1.00mm.3dshapes/PinHeader_1x01_P1.00mm_Vertical.wrl"
+      (offset (xyz 0 0 0))
+      (scale (xyz 1 1 1))
+      (rotate (xyz 0 0 0))
+    )
+  )
+  (footprint "Connector_PinHeader_1.00mm:PinHeader_1x01_P1.00mm_Vertical" (layer "F.Cu")
+    (at 138.43 80.01)
+    (descr "Through hole straight pin header, 1x01, 1.00mm pitch, single row")
+    (tags "Through hole pin header THT 1x01 1.00mm single row")
+    (property "Sheetfile" "Inputs.kicad_sch")
+    (property "Sheetname" "")
+    (attr through_hole)
+    (fp_text reference "J4" (at 0 -1.56) (layer "F.SilkS")
+      (effects (font (size 1 1) (thickness 0.15)))
+    )
+    (fp_text value "ACC OUT" (at 0 1.56) (layer "F.Fab")
+      (effects (font (size 1 1) (thickness 0.15)))
+    )
+    (fp_text user "${REFERENCE}" (at 0 0 90) (layer "F.Fab")
+      (effects (font (size 0.76 0.76) (thickness 0.114)))
+    )
+    (fp_line (start -0.695 0.685) (end 0.695 0.685) (layer "F.SilkS") (width 0.12))
+    (fp_line (start -0.695 0) (end -0.695 -0.685) (layer "F.SilkS") (width 0.12))
+    (fp_line (start 0.695 0.685) (end 0.695 0.56) (layer "F.SilkS") (width 0.12))
+    (fp_line (start -0.695 0.685) (end -0.695 0.56) (layer "F.SilkS") (width 0.12))
+    (fp_line (start 0.608276 0.685) (end 0.695 0.685) (layer "F.SilkS") (width 0.12))
+    (fp_line (start -0.695 -0.685) (end 0 -0.685) (layer "F.SilkS") (width 0.12))
+    (fp_line (start -0.695 0.685) (end -0.608276 0.685) (layer "F.SilkS") (width 0.12))
+    (fp_line (start -1.15 1) (end 1.15 1) (layer "F.CrtYd") (width 0.05))
+    (fp_line (start 1.15 1) (end 1.15 -1) (layer "F.CrtYd") (width 0.05))
+    (fp_line (start -1.15 -1) (end -1.15 1) (layer "F.CrtYd") (width 0.05))
+    (fp_line (start 1.15 -1) (end -1.15 -1) (layer "F.CrtYd") (width 0.05))
+    (fp_line (start -0.635 0.5) (end -0.635 -0.1825) (layer "F.Fab") (width 0.1))
+    (fp_line (start -0.635 -0.1825) (end -0.3175 -0.5) (layer "F.Fab") (width 0.1))
+    (fp_line (start 0.635 0.5) (end -0.635 0.5) (layer "F.Fab") (width 0.1))
+    (fp_line (start -0.3175 -0.5) (end 0.635 -0.5) (layer "F.Fab") (width 0.1))
+    (fp_line (start 0.635 -0.5) (end 0.635 0.5) (layer "F.Fab") (width 0.1))
+    (pad "1" thru_hole rect (at 0 0) (size 0.85 0.85) (drill 0.5) (layers *.Cu *.Mask)
+      (net 7 "Net-(J3-Pad3)") (pinfunction "Pin_1") (pintype "passive"))
     (model "${KICAD6_3DMODEL_DIR}/Connector_PinHeader_1.00mm.3dshapes/PinHeader_1x01_P1.00mm_Vertical.wrl"
       (offset (xyz 0 0 0))
@@
       (net 4 "Net-(J1-Pad1)") (pinfunction "Pin_1") (pintype "passive"))
     (pad "2" thru_hole oval (at 0 1) (size 0.85 0.85) (drill 0.5) (layers *.Cu *.Mask)
-      (net 2 "Net-(R1-Pad1)") (pinfunction "Pin_2") (pintype "passive"))
+      (net 2 "Net-(J1-Pad2)") (pinfunction "Pin_2") (pintype "passive"))
     (model "${KICAD6_3DMODEL_DIR}/Connector_PinHeader_1.00mm.3dshapes/PinHeader_1x02_P1.00mm_Vertical.wrl"
       (offset (xyz 0 0 0))
@@
   (segment (start 140.43 80.82) (end 141.24 80.01) (width 0.7) (layer "B.Cu") (net 5))
   (segment (start 140.43 82.55) (end 140.43 80.82) (width 0.7) (layer "B.Cu") (net 5))
+  (segment (start 138.43 82.55) (end 138.43 80.01) (width 0.7) (layer "B.Cu") (net 7))
 )

Commit message: Text
Other:
- board text added: "MongoRacing"
Changed lines of the file:
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@@
     )
+  )
+  (gr_text "MongoRacing" (at 139.7 88.9) (layer "B.Cu")
+    (effects (font (size 1.5 1.5) (thickness 0.3)) (justify mirror))
   )
   (segment (start 142.24 83.82) (end 146.05 83.82) (width 0.7) (layer "B.Cu") (net 1))

Commit message: h
Parts:
- removed J2: GROUND, Connector_PinHeader_1.00mm:PinHeader_1x02_P1.00mm_Vertical
- J1: footprint Connector_PinHeader_1.00mm:PinHeader_1x02_P1.00mm_Vertical -> Connector_PinSocket_2.54mm:PinSocket_1x02_P2.54mm_Vertical
- J3: footprint Connector_PinHeader_1.00mm:PinHeader_1x05_P1.00mm_Vertical -> Connector_PinSocket_2.54mm:PinSocket_1x05_P2.54mm_Vertical
- J4: footprint Connector_PinHeader_1.00mm:PinHeader_1x01_P1.00mm_Vertical -> Connector_PinSocket_2.54mm:PinSocket_1x01_P2.54mm_Vertical
- LDR-OUT1: footprint Connector_PinHeader_1.00mm:PinHeader_1x01_P1.00mm_Vertical -> Connector_PinHeader_2.54mm:PinHeader_1x01_P2.54mm_Vertical
- moved J1 5.68 mm to (129.5, 85.1)
- moved J4 2.84 mm to (135.9, 78.7)
- moved LDR-OUT1 1.80 mm to (143.5, 82.5)
- moved R1 1.80 mm to (135.9, 87.6)
- moved R2 1.27 mm to (147.3, 83.8)
Connections:
- J3 pad 1: Net-(J2-Pad2) -> Earth
- R2 pad 2: Net-(J2-Pad1) -> Earth
Routing:
- net Earth: track 0.00 -> 8.79 mm
- net Net-(J2-Pad1): track 3.98 -> 0.00 mm
- net Net-(J1-Pad2): track 2.81 -> 6.35 mm
- net Net-(LDR-OUT1-Pad1): track 6.35 -> 9.42 mm
- net Net-(J2-Pad2): track 2.88 -> 0.00 mm
- net Net-(J3-Pad3): track 2.54 -> 4.03 mm
- net Net-(J1-Pad1): track 1.81 -> 2.84 mm
- added copper zone on B.Cu, net Earth
