File: Kicad/Motor/Motor.kicad_pcb (KiCad board)
At the start: 2 copper layers, 7 parts, among them J1 12V, J2 PWM, J3 Motor 12V, J4 Motor Ground, J5 Ground, Q1 TIP120

Commit message: Update
Parts:
- removed J1: 12V, Connector_PinHeader_1.00mm:PinHeader_1x01_P1.00mm_Vertical
- removed J2: PWM, Connector_PinHeader_1.00mm:PinHeader_1x01_P1.00mm_Vertical
- removed J3: Motor 12V, Connector_PinHeader_1.00mm:PinHeader_1x01_P1.00mm_Vertical
- removed J4: Motor Ground, Connector_PinHeader_1.00mm:PinHeader_1x01_P1.00mm_Vertical
- removed J5: Ground, Connector_PinHeader_1.00mm:PinHeader_1x01_P1.00mm_Vertical
- added M1: M 12V og M Gorund, Connector_PinHeader_1.00mm:PinHeader_1x02_P1.00mm_Vertical, F.Cu at (153.7, 91.4)
- added PWM-12V1: PWM og 12V, Connector_PinHeader_1.00mm:PinHeader_1x02_P1.00mm_Vertical, F.Cu at (148.6, 91.4)
- added TIP-G1: Ground, Connector_PinHeader_1.00mm:PinHeader_1x01_P1.00mm_Vertical, F.Cu at (151.1, 92.7)
- moved R1 17.0 mm to (146.1, 94.0), turned to -90 degrees
- moved Q1 12.5 mm to (151.1, 101.6), turned to 90 degrees
Routing:
- net Net-(Q1-Pad2): track 0.00 -> 7.67 mm
- net Net-(Q1-Pad1): track 0.00 -> 5.08 mm
- net Net-(PWM-12V1-Pad2): track 0.00 -> 4.08 mm
- net Net-(TIP-G1-Pad1): track 0.00 -> 3.81 mm
- net Net-(R1-Pad1): track 0.00 -> 3.59 mm

Commit message: Text
Other:
- board text added: "MongoRacing"
Changed lines of the file:
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@@
     )
+  )
+  (gr_text "MongoRacing" (at 143.51 96.52 90) (layer "B.Cu")
+    (effects (font (size 1.5 1.5) (thickness 0.3)) (justify mirror))
   )
   (segment (start 148.59 91.44) (end 146.05 93.98) (width 0.7) (layer "B.Cu") (net 1))

Commit message: h
Parts:
- M1, PWM-12V1: footprint Connector_PinHeader_1.00mm:PinHeader_1x02_P1.00mm_Vertical -> Connector_PinSocket_2.54mm:PinSocket_1x02_P2.54mm_Vertical
- TIP-G1: footprint Connector_PinHeader_1.00mm:PinHeader_1x01_P1.00mm_Vertical -> Connector_PinSocket_2.54mm:PinSocket_1x01_P2.54mm_Vertical
- moved PWM-12V1 3.59 mm to (146.1, 88.9)
- moved TIP-G1 1.27 mm to (151.1, 91.4)
Connections:
- net Net-(TIP-G1-Pad1) renamed Earth
Routing:
- net Net-(M1-Pad1): track 4.08 -> 10.6 mm
- net Net-(M1-Pad2): track 7.67 -> 6.13 mm
- net Net-(PWM-12V1-Pad1): track 3.59 -> 5.08 mm
- net Earth: track 3.81 -> 5.08 mm
- added copper zone on B.Cu, net Earth
