File: Kicad/Power/Power.kicad_pcb (KiCad board)
At the start: 2 copper layers, 4 parts, among them U1 L7805

Commit message: Update
Routing:
- net Net-(Ground1-Pad1): track 0.00 -> 9.65 mm
- net Net-(U1-Pad3): track 0.00 -> 7.57 mm
- net Net-(12V1-Pad1): track 0.00 -> 6.72 mm
Changed lines of the file:
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@@
   )
   (setup
+    (stackup
+      (layer "F.SilkS" (type "Top Silk Screen"))
+      (layer "F.Paste" (type "Top Solder Paste"))
+      (layer "F.Mask" (type "Top Solder Mask") (thickness 0.01))
+      (layer "F.Cu" (type "copper") (thickness 0.035))
+      (layer "dielectric 1" (type "core") (thickness 1.51) (material "FR4") (epsilon_r 4.5) (loss_tangent 0.02))
+      (layer "B.Cu" (type "copper") (thickness 0.035))
+      (layer "B.Mask" (type "Bottom Solder Mask") (thickness 0.01))
+      (layer "B.Paste" (type "Bottom Solder Paste"))
+      (layer "B.SilkS" (type "Bottom Silk Screen"))
+      (copper_finish "None")
+      (dielectric_constraints no)
+    )
     (pad_to_mask_clearance 0)
     (pcbplotparams
@@
     )
   )
+  (segment (start 131.62 56.47) (end 131.68 56.41) (width 0.7) (layer "B.Cu") (net 1))
+  (segment (start 132.62 60.96) (end 133.62 60.96) (width 0.7) (layer "B.Cu") (net 1))
+  (segment (start 131.62 60.96) (end 131.62 56.47) (width 0.7) (layer "B.Cu") (net 1))
+  (segment (start 133.62 60.96) (end 134.62 60.96) (width 0.7) (layer "B.Cu") (net 1))
+  (segment (start 131.62 60.96) (end 132.62 60.96) (width 0.7) (layer "B.Cu") (net 1))
+  (segment (start 120.38 56.81) (end 120.78 56.41) (width 0.7) (layer "B.Cu") (net 2))
+  (segment (start 119.38 60.96) (end 120.38 60.96) (width 0.7) (layer "B.Cu") (net 2))
+  (segment (start 120.38 60.96) (end 120.38 56.81) (width 0.7) (layer "B.Cu") (net 2))
+  (segment (start 121.38 60.96) (end 120.38 60.96) (width 0.7) (layer "B.Cu") (net 2))
+  (segment (start 126.46 60.96) (end 126.46 56.64) (width 0.7) (layer "B.Cu") (net 3))
+  (segment (start 128.46 60.96) (end 129.46 60.96) (width 0.7) (layer "B.Cu") (net 3))
+  (segment (start 126.46 56.64) (end 126.23 56.41) (width 0.7) (layer "B.Cu") (net 3))
+  (segment (start 126.46 60.96) (end 127.46 60.96) (width 0.7) (layer "B.Cu") (net 3))
+  (segment (start 124.46 60.96) (end 125.46 60.96) (width 0.7) (layer "B.Cu") (net 3))
+  (segment (start 125.46 60.96) (end 126.46 60.96) (width 0.7) (layer "B.Cu") (net 3))
+  (segment (start 127.46 60.96) (end 128.46 60.96) (width 0.7) (layer "B.Cu") (net 3))
 )

Commit message: Text
Other:
- board text added: "MongoRacing"
Changed lines of the file:
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@@
     )
+  )
+  (gr_text "MongoRacing" (at 125.73 52.07) (layer "B.Cu")
+    (effects (font (size 1.5 1.5) (thickness 0.3)) (justify mirror))
   )
   (segment (start 131.62 56.47) (end 131.68 56.41) (width 0.7) (layer "B.Cu") (net 1))

Commit message: h
Parts:
- 12V1: footprint Connector_PinHeader_1.00mm:PinHeader_1x03_P1.00mm_Vertical -> Connector_PinSocket_2.54mm:PinSocket_1x03_P2.54mm_Vertical
- 5V1: footprint Connector_PinHeader_1.00mm:PinHeader_1x04_P1.00mm_Vertical -> Connector_PinHeader_2.54mm:PinHeader_1x04_P2.54mm_Vertical
- Ground1: footprint Connector_PinHeader_1.00mm:PinHeader_1x06_P1.00mm_Vertical -> Connector_PinHeader_2.54mm:PinHeader_1x06_P2.54mm_Vertical
- moved Ground1 9.67 mm to (120.7, 52.1)
- moved 5V1 2.84 mm to (135.9, 63.5), turned to 180 degrees
- moved 12V1 1.80 mm to (120.7, 62.2)
Connections:
- net Net-(Ground1-Pad1) renamed Earth
Routing:
- net Earth: track 9.65 -> 17.6 mm
- net Net-(12V1-Pad1): track 6.72 -> 11.0 mm
- net Net-(5V1-Pad1): track 7.57 -> 9.59 mm
- added copper zone on B.Cu, net Earth
