File: Kicad/Power/Power.kicad_sch (KiCad schematic)
At the start: 4 parts, among them U1 L7805

Commit message: h
Parts:
- 12V1: value Conn_01x03_Female -> (none); footprint Connector_PinHeader_1.00mm:PinHeader_1x03_P1.00mm_Vertical -> (none)
- 5V1: value Conn_01x04_Female -> (none); footprint Connector_PinHeader_1.00mm:PinHeader_1x04_P1.00mm_Vertical -> (none)
- Ground1: value Conn_01x06_Female -> (none); footprint Connector_PinHeader_1.00mm:PinHeader_1x06_P1.00mm_Vertical -> (none)
Connections:
- net Earth: now reaches Ground1.1 (Pin_1), Ground1.2 (Pin_2), Ground1.3 (Pin_3), Ground1.4 (Pin_4), Ground1.5 (Pin_5), Ground1.6 (Pin_6), U1.2 (GND)
Changed lines of the file:
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@@
   (junction (at 110.49 82.55) (diameter 0) (color 0 0 0 0)
+  )
+  (junction (at 121.92 86.36) (diameter 0) (color 0 0 0 0)
   )
   (junction (at 110.49 86.36) (diameter 0) (color 0 0 0 0)
@@
       (effects (font (size 1.27 1.27)) (justify left))
     )
-    (property "Value" "Conn_01x04_Female" (id 1) (at 140.97 77.4699 0)
+    (property "Value" "" (id 1) (at 140.97 77.4699 0)
       (effects (font (size 1.27 1.27)) (justify left) hide)
     )
-    (property "Footprint" "Connector_PinHeader_1.00mm:PinHeader_1x04_P1.00mm_Vertical" (id 2) (at 139.7 74.93 0)
+    (property "Footprint" "" (id 2) (at 139.7 74.93 0)
       (effects (font (size 1.27 1.27)) hide)
     )
@@
     (in_bom yes) (on_board yes) (fields_autoplaced)
     (property "Reference" "Ground1" (id 0) (at 106.045 77.47 0))
-    (property "Value" "Conn_01x06_Female" (id 1) (at 106.045 77.47 0)
+    (property "Value" "" (id 1) (at 106.045 77.47 0)
       (effects (font (size 1.27 1.27)) hide)
     )
-    (property "Footprint" "Connector_PinHeader_1.00mm:PinHeader_1x06_P1.00mm_Vertical" (id 2) (at 105.41 87.63 0)
+    (property "Footprint" "" (id 2) (at 105.41 87.63 0)
       (effects (font (size 1.27 1.27)) hide)
     )
@@
     (in_bom yes) (on_board yes) (fields_autoplaced)
     (property "Reference" "12V1" (id 0) (at 106.045 67.31 0))
-    (property "Value" "Conn_01x03_Female" (id 1) (at 106.045 67.31 0)
+    (property "Value" "" (id 1) (at 106.045 67.31 0)
       (effects (font (size 1.27 1.27)) hide)
     )
-    (property "Footprint" "Connector_PinHeader_1.00mm:PinHeader_1x03_P1.00mm_Vertical" (id 2) (at 105.41 72.39 0)
+    (property "Footprint" "" (id 2) (at 105.41 72.39 0)
       (effects (font (size 1.27 1.27)) hide)
     )
@@
     (pin "2")
     (pin "3")
+  )
+  (symbol (lib_id "power:Earth") (at 121.92 86.36 0) (unit 1)
+    (in_bom yes) (on_board yes) (fields_autoplaced)
+    (property "Reference" "#PWR?" (id 0) (at 121.92 92.71 0)
+      (effects (font (size 1.27 1.27)) hide)
+    )
+    (property "Value" "Earth" (id 1) (at 121.92 90.17 0)
+      (effects (font (size 1.27 1.27)) hide)
+    )
+    (property "Footprint" "" (id 2) (at 121.92 86.36 0)
+      (effects (font (size 1.27 1.27)) hide)
+    )
+    (property "Datasheet" "~" (id 3) (at 121.92 86.36 0)
+      (effects (font (size 1.27 1.27)) hide)
+    )
+    (pin "1")
   )
   (symbol (lib_id "Regulator_Linear:L7805") (at 121.92 76.2 0) (unit 1)
@@
   )
   (symbol_instances
+    (path "/92563de1-61c4-4e3f-8603-96474790934f"
+      (reference "#PWR?") (unit 1) (value "Earth") (footprint "")
+    )
     (path "/019be7a5-8b04-48f6-a390-7528e4489879"
-      (reference "5V1") (unit 1) (value "Conn_01x04_Female") (footprint "Connector_PinHeader_1.00mm:PinHeader_1x04_P1.00mm_Vertical")
+      (reference "5V1") (unit 1) (value "Conn_01x04_Female") (footprint "Connector_PinHeader_2.54mm:PinHeader_1x04_P2.54mm_Vertical")
     )
     (path "/751a72d0-6d44-4212-8f4e-176cab5fa2ec"
-      (reference "12V1") (unit 1) (value "Conn_01x03_Female") (footprint "Connector_PinHeader_1.00mm:PinHeader_1x03_P1.00mm_Vertical")
+      (reference "12V1") (unit 1) (value "Conn_01x03_Female") (footprint "Connector_PinSocket_2.54mm:PinSocket_1x03_P2.54mm_Vertical")
     )
     (path "/10d96478-cd94-400b-8b17-5e4d4aa73dc4"
-      (reference "Ground1") (unit 1) (value "Conn_01x06_Female") (footprint "Connector_PinHeader_1.00mm:PinHeader_1x06_P1.00mm_Vertical")
+      (reference "Ground1") (unit 1) (value "Conn_01x06_Female") (footprint "Connector_PinHeader_2.54mm:PinHeader_1x06_P2.54mm_Vertical")
     )
     (path "/b4d50de9-8498-49c0-bb18-a5f3cbd8c5ba"
