File: Kicad/Samlet PCB/Samlet Racerbil.kicad_pcb (KiCad board)
At the start: 2 copper layers, 11 parts, among them J1 Pickit Forbindelse, J2 LED, J5 Conn_01x05_Female, Q1 IRL1404, U1 L7805, U2 PIC16F684-IP

Commit message: update
Parts:
- moved J5 35.7 mm to (147.3, 88.9)
- moved U1 34.5 mm to (152.4, 94.0), turned to 90 degrees
- moved J1 34.2 mm to (124.5, 100.3), turned to 180 degrees
- moved U2 26.9 mm to (142.2, 64.8), turned to -90 degrees
- moved Q1 18.1 mm to (119.4, 83.8), turned to 90 degrees
- moved R1 16.3 mm to (121.9, 63.5), turned to -90 degrees
- moved R3 15.3 mm to (152.4, 68.6), turned to 180 degrees
- moved R2 14.2 mm to (152.4, 83.8)
- moved J2 10.2 mm to (147.3, 82.5)
- moved Power1 3.81 mm to (135.9, 61.0)
Routing:
- net 5V: track 0.00 -> 100.3 mm
- net ACC: track 0.00 -> 90.8 mm
- net 12V: track 11.4 -> 75.8 mm
- net Net-(J1-Pad6): track 0.00 -> 45.3 mm
- net Net-(J1-Pad2): track 0.00 -> 36.5 mm
- net Net-(J1-Pad3): track 0.00 -> 34.4 mm
- net LDR: track 3.82 -> 35.7 mm
- net Lys: track 0.00 -> 28.6 mm
- net Net-(Q1-Pad1): track 6.48 -> 16.3 mm
- net PWM: track 11.2 -> 13.5 mm
- net Net-(JMotor1-Pad2): track 18.0 -> 16.1 mm
Other:
- board text added: "MongoRacing"

Commit message: Update Samlet Racerbil.kicad_pcb
Routing:
- added copper zone on B.Cu, net Ground
- added copper zone on F.Cu, net Ground
Other:
- board text added: "MongoRacing Chipset 2000X"
- board text removed: "MongoRacing"
Changed lines of the file:
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@@
     )
   )
-  (gr_text "MongoRacing\n" (at 119.38 93.98 90) (layer "F.Cu")
+  (gr_text "MongoRacing\nChipset 2000X" (at 118.11 95.25 90) (layer "F.Cu")
     (effects (font (size 1.2 1.2) (thickness 0.25)))
   )
@@
   (segment (start 152.4 73.66) (end 152.4 68.58) (width 0.7) (layer "B.Cu") (net 17))
   (segment (start 151.13 66.04) (end 152.4 67.31) (width 0.7) (layer "B.Cu") (net 17))
+  (zone (net 4) (net_name "Ground") (layers F&B.Cu) (hatch edge 0.508)
+    (connect_pads (clearance 0.508))
+    (min_thickness 0.254) (filled_areas_thickness no)
+    (fill yes (thermal_gap 0.508) (thermal_bridge_width 0.508))
+    (polygon
+      (pts
+        (xy 156.21 102.87)
+        (xy 115.57 102.87)
+        (xy 115.57 58.42)
+        (xy 156.21 58.42)
+      )
+    )
+  )
 )

Commit message: Capacitor
Parts:
- added C1: C, Capacitor_THT:CP_Radial_D7.5mm_P2.50mm, F.Cu at (147.3, 61.0)

Commit message: h
Parts:
- removed J2: LED, Connector_PinHeader_2.54mm:PinHeader_1x04_P2.54mm_Vertical
- moved JMotor1 31.4 mm to (143.5, 106.7)
- moved R1 30.7 mm to (125.7, 94.0)
- moved J1 29.0 mm to (142.2, 77.5), turned to -90 degrees
- moved J5 25.0 mm to (124.5, 78.7)
- moved Q1 23.3 mm to (130.8, 104.1), turned to 0 degrees
- moved Power1 21.8 mm to (148.6, 78.7)
- moved R3 21.7 mm to (144.8, 88.9), turned to 90 degrees
- moved U2 21.2 mm to (130.8, 82.6), turned to 0 degrees
- moved C1 19.3 mm to (154.9, 78.7), turned to -90 degrees
- moved R2 15.3 mm to (153.7, 99.1), turned to 180 degrees
- moved U1 6.36 mm to (152.7, 87.6), turned to -90 degrees
Routing:
- net ACC: track 90.8 -> 0.00 mm
- net Lys: track 28.6 -> 0.00 mm
- net Net-(J1-Pad6): track 45.3 -> 16.8 mm
- net Net-(J1-Pad3): track 34.4 -> 10.3 mm
- net Net-(J1-Pad2): track 36.5 -> 12.9 mm
- net 12V: track 75.8 -> 56.9 mm
- net LDR: track 35.7 -> 17.3 mm
- net 5V: track 100.3 -> 87.7 mm
- net Net-(Q1-Pad1): track 16.3 -> 5.08 mm
- net PWM: track 13.5 -> 5.65 mm
- net Net-(JMotor1-Pad2): track 16.1 -> 10.2 mm
- removed copper zone on F.Cu, net Ground
Other:
- board text removed: "MongoRacing Chipset 2000X"
